Commit message: Added camera... can't change color of it...

File: catkin_ws/src/udacity_bot/urdf/udacity_bot.xacro (robot description, xacro)
@@ -125,3 +125,35 @@
         </collision>
     </link>
+    <!-- *********  Camera ******************************** -->
+    <joint name="camera_joint" type="fixed">
+        <origin xyz="0.2 0 0" rpy="0 0 0"/>
+        <child link="camera"/>
+        <parent link="chassis"/>
+    </joint>
+    <link name='camera'>
+        <inertial>
+            <mass value="0.1"/>
+            <origin xyz="0 0 0" rpy="0 0 0"/>
+            <inertia
+                    ixx="1e-6" ixy="0" ixz="0"
+                    iyy="1e-6" iyz="0"
+                    izz="1e-6"
+            />
+        </inertial>
+        <visual>
+            <geometry>
+                <box size="0.05 0.05 0.05"/>
+            </geometry>
+            <origin xyz="0 0 0" rpy="0 0 0"/>
+            <material name="blue">
+                <color rgba="0 0 1 1"/>
+            </material>
+        </visual>
+        <collision>
+            <geometry>
+                <box size="0.05 0.05 0.05"/>
+            </geometry>
+            <origin xyz="0 0 0" rpy="0 0 0"/>
+        </collision>
+    </link>
 </robot>

Commit message: Added koyuko to robot model

File: catkin_ws/src/udacity_bot/urdf/udacity_bot.xacro (robot description, xacro)
@@ -29,4 +29,7 @@
                 <box size=".4 .2 .1"/>
             </geometry>
+            <material name="white_seethru">
+                <color rgba="1 1 1 0.1"/>
+            </material>
         </visual>
         <collision name='back_caster_collision'>
@@ -157,3 +160,32 @@
         </collision>
     </link>
+    <!-- *********  Laser Rangefinder ******************************** -->
+    <joint type="fixed" name="hokuyo_joint">
+        <origin xyz="0.15 0 0.1" rpy="0 0 0"/>
+        <child link="hokuyo"/>
+        <parent link="chassis"/>
+    </joint>
+    <link name="hokuyo">
+        <inertial>
+            <mass value="0.1"/>
+            <origin xyz="0 0 0" rpy="0 0 0"/>
+            <inertia
+                    ixx="1e-6" ixy="0" ixz="0"
+                    iyy="1e-6" iyz="0"
+                    izz="1e-6"
+            />
+        </inertial>
+        <visual>
+            <geometry>
+                <mesh filename="package://udacity_bot/meshes/hokuyo.dae"/>
+            </geometry>
+            <origin xyz="0 0 0" rpy="0 0 0"/>
+        </visual>
+        <collision>
+            <geometry>
+                <box size="0.1 0.1 0.1"/>
+            </geometry>
+            <origin xyz="0 0 0" rpy="0 0 0"/>
+        </collision>
+    </link>
 </robot>

Commit message: Add supplied .gazebo file

File: catkin_ws/src/udacity_bot/urdf/udacity_bot.xacro (robot description, xacro)
@@ -1,4 +1,5 @@
 <?xml version='1.0'?>
 <robot name="udacity_bot" xmlns:xacro="http://www.ros.org/wiki/xacro">
+    <xacro:include filename="$(find udacity_bot)/urdf/udacity_bot.gazebo" />
     <link name="robot_footprint"></link>
     <joint name="robot_footprint_joint" type="fixed">
@@ -29,7 +30,4 @@
                 <box size=".4 .2 .1"/>
             </geometry>
-            <material name="white_seethru">
-                <color rgba="1 1 1 0.1"/>
-            </material>
         </visual>
         <collision name='back_caster_collision'>

Commit message: Change ciel bot to cylinder chassis

File: catkin_ws/src/udacity_bot/urdf/udacity_bot.xacro (robot description, xacro)
@@ -58,5 +58,5 @@
     <!-- *********  Left Wheel ******************************** -->
     <joint name="left_wheel_hinge" type="continuous">
-        <origin xyz="0 0.15 0" rpy="0 0 0"/>
+        <origin xyz="0 0.25 0" rpy="0 0 0"/>
         <child link="left_wheel"/>
         <parent link="chassis"/>
@@ -93,5 +93,5 @@
     <!-- *********  Right Wheel ******************************** -->
     <joint name="right_wheel_hinge" type="continuous">
-        <origin xyz="0 -0.15 0" rpy="0 0 0"/>
+        <origin xyz="0 -0.25 0" rpy="0 0 0"/>
         <child link="right_wheel"/>
         <parent link="chassis"/>
@@ -128,5 +128,5 @@
     <!-- *********  Camera ******************************** -->
     <joint name="camera_joint" type="fixed">
-        <origin xyz="0.2 0 0" rpy="0 0 0"/>
+        <origin xyz="0.25 0 0" rpy="0 0 0"/>
         <child link="camera"/>
         <parent link="chassis"/>
@@ -160,5 +160,5 @@
     <!-- *********  Laser Rangefinder ******************************** -->
     <joint type="fixed" name="hokuyo_joint">
-        <origin xyz="0.15 0 0.1" rpy="0 0 0"/>
+        <origin xyz="0.0 0 0.1" rpy="0 0 0"/>
         <child link="hokuyo"/>
         <parent link="chassis"/>

File: catkin_ws/src/udacity_bot/urdf/udacity_bot_ciel.xacro (robot description, xacro)
@@ -22,5 +22,5 @@
             <origin xyz="0 0 0" rpy=" 0 0 0"/>
             <geometry>
-                <box size=".4 .2 .1"/>
+                <cylinder radius="0.2" length="0.15"/>
             </geometry>
         </collision>
@@ -28,5 +28,5 @@
             <origin xyz="0 0 0" rpy=" 0 0 0"/>
             <geometry>
-                <box size=".4 .2 .1"/>
+                <cylinder radius="0.2" length="0.15"/>
             </geometry>
             <material name="purple">
@@ -35,5 +35,5 @@
         </visual>
         <collision name='back_caster_collision'>
-            <origin xyz="-0.15 0 -0.05" rpy=" 0 0 0"/>
+            <origin xyz="-0.15 0 -0.1" rpy=" 0 0 0"/>
             <geometry>
                 <sphere radius="0.0499"/>
@@ -41,5 +41,5 @@
         </collision>
         <visual name='back_caster_visual'>
-            <origin xyz="-0.15 0 -0.05" rpy=" 0 0 0"/>
+            <origin xyz="-0.15 0 -0.1" rpy=" 0 0 0"/>
             <geometry>
                 <sphere radius="0.05"/>
@@ -47,5 +47,5 @@
         </visual>
         <collision name='front_caster_collision'>
-            <origin xyz="0.15 0 -0.05" rpy=" 0 0 0"/>
+            <origin xyz="0.15 0 -0.1" rpy=" 0 0 0"/>
             <geometry>
                 <sphere radius="0.0499"/>
@@ -53,5 +53,5 @@
         </collision>
         <visual name='front_caster_visual'>
-            <origin xyz="0.15 0 -0.05" rpy=" 0 0 0"/>
+            <origin xyz="0.15 0 -0.1" rpy=" 0 0 0"/>
             <geometry>
                 <sphere radius="0.05"/>
@@ -61,5 +61,5 @@
     <!-- *********  Left Wheel ******************************** -->
     <joint name="left_wheel_hinge" type="continuous">
-        <origin xyz="0.15 0.15 0" rpy="0 0 0"/>
+        <origin xyz="0 0.2 -0.05" rpy="0 0 0"/>
         <child link="left_wheel"/>
         <parent link="chassis"/>
@@ -96,5 +96,5 @@
     <!-- *********  Right Wheel ******************************** -->
     <joint name="right_wheel_hinge" type="continuous">
-        <origin xyz="0.15 -0.15 0" rpy="0 0 0"/>
+        <origin xyz="0 -0.2 -0.05" rpy="0 0 0"/>
         <child link="right_wheel"/>
         <parent link="chassis"/>
@@ -131,5 +131,5 @@
     <!-- *********  Camera ******************************** -->
     <joint name="camera_joint" type="fixed">
-        <origin xyz="0.2 0 0" rpy="0 0 0"/>
+        <origin xyz="0.0 0 0" rpy="0 0 0"/>
         <child link="camera"/>
         <parent link="chassis"/>
@@ -163,5 +163,5 @@
     <!-- *********  Laser Rangefinder ******************************** -->
     <joint type="fixed" name="hokuyo_joint">
-        <origin xyz="0.15 0 0.1" rpy="0 0 0"/>
+        <origin xyz="0.0 0 0.1" rpy="0 0 0"/>
         <child link="hokuyo"/>
         <parent link="chassis"/>

Commit message: Fix original bot laser position

File: catkin_ws/src/udacity_bot/urdf/udacity_bot.xacro (robot description, xacro)
@@ -58,5 +58,5 @@
     <!-- *********  Left Wheel ******************************** -->
     <joint name="left_wheel_hinge" type="continuous">
-        <origin xyz="0 0.25 0" rpy="0 0 0"/>
+        <origin xyz="0 0.15 0" rpy="0 0 0"/>
         <child link="left_wheel"/>
         <parent link="chassis"/>
@@ -93,5 +93,5 @@
     <!-- *********  Right Wheel ******************************** -->
     <joint name="right_wheel_hinge" type="continuous">
-        <origin xyz="0 -0.25 0" rpy="0 0 0"/>
+        <origin xyz="0 -0.15 0" rpy="0 0 0"/>
         <child link="right_wheel"/>
         <parent link="chassis"/>
@@ -160,5 +160,5 @@
     <!-- *********  Laser Rangefinder ******************************** -->
     <joint type="fixed" name="hokuyo_joint">
-        <origin xyz="0.0 0 0.1" rpy="0 0 0"/>
+        <origin xyz="0.15 0 0.1" rpy="0 0 0"/>
         <child link="hokuyo"/>
         <parent link="chassis"/>
